Commit message: [FIX] fix urdf bug

File: src/robotsky_description/urdf/robotsky_wq.urdf (robot description, URDF)
Before this commit: robot robotsky_wq, 17 links, 16 joints
Links:
- link LB_Hip_Link: geometry collision mesh filename=package://robotsky_description/meshes/robotsky_wq/LB_Hip_Li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; visual mesh filename=package://robotsky_description/meshes/robotsky_wq/LB_Hip_Li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
- link LB_Knee_Link: geometry collision mesh filename=package://robotsky_description/meshes/robotsky_wq/LB_Knee_L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; visual mesh filename=package://robotsky_description/meshes/robotsky_wq/LB_Knee_L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
- link LB_Roll_Link: geometry collision mesh filename=package://robotsky_description/meshes/robotsky_wq/LB_Roll_L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; visual mesh filename=package://robotsky_description/meshes/robotsky_wq/LB_Roll_L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
- link LB_Wheel_Link: geometry collision cylinder length=0.035 radius=0.075; visual mesh filename=package://robotsky_description/meshes/robotsky_wq/LB_Wheel_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
- link LF_Hip_Link: geometry collision mesh filename=package://robotsky_description/meshes/robotsky_wq/LF_Hip_Li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; visual mesh filename=package://robotsky_description/meshes/robotsky_wq/LF_Hip_Li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
- link LF_Knee_Link: geometry collision mesh filename=package://robotsky_description/meshes/robotsky_wq/LF_Knee_L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; visual mesh filename=package://robotsky_description/meshes/robotsky_wq/LF_Knee_L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
- link LF_Roll_Link: geometry collision mesh filename=package://robotsky_description/meshes/robotsky_wq/LF_Roll_L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; visual mesh filename=package://robotsky_description/meshes/robotsky_wq/LF_Roll_L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
- link LF_Wheel_Link: geometry collision cylinder length=0.035 radius=0.075; visual mesh filename=package://robotsky_description/meshes/robotsky_wq/LF_Wheel_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
- link RB_Hip_Link: geometry collision mesh filename=package://robotsky_description/meshes/robotsky_wq/RB_Hip_Li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; visual mesh filename=package://robotsky_description/meshes/robotsky_wq/RB_Hip_Li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
- link RB_Knee_Link: geometry collision mesh filename=package://robotsky_description/meshes/robotsky_wq/RB_Knee_L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; visual mesh filename=package://robotsky_description/meshes/robotsky_wq/RB_Knee_L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
- link RB_Roll_Link: geometry collision mesh filename=package://robotsky_description/meshes/robotsky_wq/RB_Roll_L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; visual mesh filename=package://robotsky_description/meshes/robotsky_wq/RB_Roll_L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
- link RB_Wheel_Link: geometry collision cylinder length=0.035 radius=0.075; visual mesh filename=package://robotsky_description/meshes/robotsky_wq/RB_Wheel_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
- link RF_Hip_Link: geometry collision mesh filename=package://robotsky_description/meshes/robotsky_wq/RF_Hip_Li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; visual mesh filename=package://robotsky_description/meshes/robotsky_wq/RF_Hip_Li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
- link RF_Knee_Link: geometry collision mesh filename=package://robotsky_description/meshes/robotsky_wq/RF_Knee_L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; visual mesh filename=package://robotsky_description/meshes/robotsky_wq/RF_Knee_L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
- link RF_Roll_Link: geometry collision mesh filename=package://robotsky_description/meshes/robotsky_wq/RF_Roll_L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; visual mesh filename=package://robotsky_description/meshes/robotsky_wq/RF_Roll_L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
- link RF_Wheel_Link: geometry collision cylinder length=0.035 radius=0.075; visual mesh filename=package://robotsky_description/meshes/robotsky_wq/RF_Wheel_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
- link base_link: geometry collision mesh filename=package://robotsky_description/meshes/robotsky_wq/base_link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; visual mesh filename=package://robotsky_description/meshes/robotsky_wq/base_link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
